Commit message: all direction movement done

File: urdf/inof_robot.urdf.xacro (robot description, xacro)
@@ -44,4 +44,7 @@
 			</inertial>
 		</link>
+		<gazebo reference="layer${level}">
+			<material>Gazebo/Red</material>
+		</gazebo>
 	</xacro:macro>
 	<xacro:macro name="support_leg" params="number x y z">

Commit message: all done

File: urdf/inof_robot.urdf.xacro (robot description, xacro)
@@ -9,5 +9,5 @@
 	<xacro:property name="casterlen" value="0.012"/>
 	<xacro:property name="casterwid" value="0.012"/>
-	<xacro:property name="casterhgt" value="0.02375"/>
+	<xacro:property name="casterhgt" value="0.025"/>
 	<xacro:property name="layerweight" value="0.0378169"/>
 	<xacro:property name="supportweight" value="0.0015127"/>
